File: hw/SmartFan.sch (KiCad schematic (older format))
At the start: 25 parts

Commit message: IMM-NRF52832 Schematic updates
Parts:
- removed Q? (x8): 2N3904, TO_SOT_Packages_THT:TO-92_Inline_Narrow_Oval, symbol Q_NPN_BCE
- removed R? (x8): 1k, Resistors_THT:R_Axial_DIN0207_L6.3mm_D2.5mm_P10.16mm_Horizontal, symbol R
- removed R? (x8): 10k, Resistors_THT:R_Axial_DIN0207_L6.3mm_D2.5mm_P10.16mm_Horizontal, symbol R
- removed U?: ESP32-DevKitC, ESP32-DevKitC:ESP32-DevKit-C, symbol ESP32-DevKitC
- added C? (x2): 10uF, symbol C
- added C?: 22uF, symbol C
- added D?: LED, symbol LED
- added J?: Fan_Conn, symbol Conn_01x06
- added J?: Relay_Conn, symbol Conn_01x06
- added J?: Conn_ARM_JTAG_SWD_20, symbol Conn_ARM_JTAG_SWD_20
- added Q? (x3): Q_PNP_BCE, symbol Q_PNP_BCE
- added R? (x3): 1K, symbol R
- added R? (x3): 10K, symbol R
- added R?: 2k, symbol R
- added R?: R, symbol R
- added R?: 3.3K, symbol R
- added U?: IMM-NRF52832, symbol IMM-NRF52832
- added U?: NCP1117ST33T3G, digikey-footprints:SOT-223, symbol NCP1117ST33T3G
Connections:
- net labels added: +3.3V
- net labels removed: +3V3
- wire segments 80 -> 61
- no-connect marks 9 -> 10
