File: hw/SmartFan.sch (KiCad schematic (older format))
At the start: 25 parts

Commit message: Hardware redesign and 1st PCB layout
Parts:
- removed Q? (x8): 2N3904, TO_SOT_Packages_THT:TO-92_Inline_Narrow_Oval, symbol Q_NPN_BCE
- removed R? (x8): 1k, Resistors_THT:R_Axial_DIN0207_L6.3mm_D2.5mm_P10.16mm_Horizontal, symbol R
- removed R? (x8): 10k, Resistors_THT:R_Axial_DIN0207_L6.3mm_D2.5mm_P10.16mm_Horizontal, symbol R
- removed U?: ESP32-DevKitC, ESP32-DevKitC:ESP32-DevKit-C, symbol ESP32-DevKitC
- added C1: 10uF, Capacitors_SMD:C_0805, symbol C
- added C2, C3: 1uF, Capacitors_SMD:C_0805, symbol C
- added C4: 0.1uF, Capacitors_SMD:C_0805, symbol C
- added D1: MBR0540T1G, digikey-footprints:SOD-123, symbol MBR0540T1G
- added D2, D3, D4: 1N4148W-7-F, digikey-footprints:SOD-123, symbol 1N4148W-7-F
- added J1: Barrel_Jack, Connectors:BARREL_JACK, symbol Barrel_Jack
- added J2: JTAG_SWD, Connectors_IDC:IDC-Header_2x10_Pitch2.54mm_Straight, symbol Conn_02x10_Odd_Even
- added J3: FAN_CONN, Connectors_Molex:Molex_MegaFit_2x02x5.70mm_Angled, symbol Conn_02x02_Counter_Clockwise
- added MOD1: BMD-300-A-R, digikey-footprints:Bluetooth_Module_BMD-300, symbol BMD-300-A-R
- added Q1, Q2, Q3: MMBT2222A-TP, digikey-footprints:SOT-23-3, symbol MMBT2222A-TP
- added Q4, Q5, Q6: MMBT2222A-7-F, digikey-footprints:SOT-23-3, symbol MMBT2222A-7-F
- added R1, R10, R11, R12, R13, R14, R15, R2, R5, R7, R8, R9: 1k, Resistors_SMD:R_0805, symbol R
- added R3, R4, R6: 10k, Resistors_SMD:R_0805, symbol R
- added RLY1, RLY2, RLY3: G5LE-14_DC5, digikey-footprints:Relay_THT_G5LE-14, symbol G5LE-14_DC5
- added U1: L7805CV, digikey-footprints:SOT-23-3, symbol L7805CV
- added U2, U3, U4: LTV-816S-TA1, digikey-footprints:SMD-4_4.6x7.62mm_P2.54mm, symbol LTV-816S-TA1
Connections:
- net labels added: +3.3V, 120VAC_IN, HI_SPD_120VAC, HI_SPD_EN, LO_SPD_120VAC, LO_SPD_EN, MED_SPD_120VAC, MED_SPD_EN, SWCLK, SWDIO, ~RESET
- net labels removed: +3V3
- wire segments 80 -> 141
- no-connect marks 9 -> 38

Commit message: Updated schematics and PCB
Parts:
- removed R13, R14: 1k, Resistors_SMD:R_0805, symbol R
- added C5, C6: 1uF, Capacitors_SMD:C_0805, symbol C
- added C7: 0.1uF, Capacitors_SMD:C_0805, symbol C
- added D5: MBR0540T1G, digikey-footprints:SOD-123, symbol MBR0540T1G
- added J3: BTLE_LED_Conn, 640456-2:TE_640456-2, symbol Conn_01x02
- added J4: ANT_LED_Conn, 640456-2:TE_640456-2, symbol Conn_01x02
- added J5: RGB_LED_Conn, 640456-4:TE_640456-4, symbol Conn_01x04
- added J6: PB_Conn, 640456-2:TE_640456-2, symbol Conn_01x02
- added Q1, Q2: MMBT2222A-7-F, digikey-footprints:SOT-23-3, symbol MMBT2222A-7-F
- added R1, R3: 220, Resistors_SMD:R_0805, symbol R
- added R11: 10k, Resistors_SMD:R_0805, symbol R
- added R19, R2, R20, R4: 330, Resistors_SMD:R_0805, symbol R
- added U5: LD1117S33CTR, digikey-footprints:SOT-223, symbol LD1117S33CTR
- R15: value 1k -> 330
- renumbered J3 to J7, Q1 to Q3, Q2 to Q4, Q3 to Q5, Q4 to Q6, Q5 to Q7, Q6 to Q8, R6 to R10, R7 to R12, R8 to R13, R9 to R14, R10 to R16, R11 to R17, R12 to R18, R1 to R5, R2 to R6, R3 to R7, R4 to R8, R5 to R9
Connections:
- net labels added: +9V, ANT_LED, BTLE_LED, RGB_LED_G, RGB_LED_R, RGB_LED_Y, SPD_CTRL_PB
- wire segments 141 -> 186
- no-connect marks 38 -> 36
Other:
- note added: "3.3v Power Regulator"
- note added: "5v Power Regulator"
- note added: "7-12vdc Power In"
- note added: "ANT+ Indicator LED (Red)"
- note added: "BTLE Indicator LED (Blue)"
- note added: "Fan Speed Control Pushbutton\n(Momentary)"
- note added: "Fan Speed Indicator LED"
- note added: "Power Flags"
- note added: "SWD Programming Port"

Commit message: many updates
Parts:
- removed J3: BTLE_LED_Conn, 640456-2:TE_640456-2, symbol Conn_01x02
- removed J4: ANT_LED_Conn, 640456-2:TE_640456-2, symbol Conn_01x02
- removed J5: RGB_LED_Conn, 640456-4:TE_640456-4, symbol Conn_01x04
- removed J6: PB_Conn, 640456-2:TE_640456-2, symbol Conn_01x02
- removed R11: 10k, Resistors_SMD:R_0805, symbol R
- added D? (x2): 1N914BTR, digikey-footprints:DO-35, symbol SmartFan-rescue:1N914BTR
- added Q? (x6): 2N3904, TO_SOT_Packages_THT:TO-92_Molded_Narrow, symbol SmartFan-rescue:2N3904
- added R? (x2): 10k, symbol SmartFan-rescue:R
- added R? (x4): 4.7k, symbol SmartFan-rescue:R
- added R? (x4): 330, symbol SmartFan-rescue:R
- added R? (x4): R, symbol SmartFan-rescue:R
- added R? (x3): 220, symbol SmartFan-rescue:R
- C1, C2, C3, C4, C5, C6, C7: symbol C -> SmartFan-rescue:C
- D1, D5: symbol MBR0540T1G -> SmartFan-rescue:MBR0540T1G
- D2, D3, D4: symbol 1N4148W-7-F -> SmartFan-rescue:1N4148W-7-F
- J1: symbol Barrel_Jack -> SmartFan-rescue:Barrel_Jack
- J2: symbol Conn_02x10_Odd_Even -> SmartFan-rescue:Conn_02x10_Odd_Even
- J7: symbol Conn_02x02_Counter_Clockwise -> SmartFan-rescue:Conn_02x02_Counter_Clockwise
- MOD1: symbol BMD-300-A-R -> SmartFan-rescue:BMD-300-A-R
- Q1, Q2, Q6, Q7, Q8: symbol MMBT2222A-7-F -> SmartFan-rescue:MMBT2222A-7-F
- Q3, Q4, Q5: symbol MMBT2222A-TP -> SmartFan-rescue:MMBT2222A-TP
- R1, R10, R12, R13, R14, R15, R16, R17, R18, R19, R2, R20, R3, R4, R5, R6, R7, R8, R9: symbol R -> SmartFan-rescue:R
- RLY1, RLY2, RLY3: symbol G5LE-14_DC5 -> SmartFan-rescue:G5LE-14_DC5
- U1: symbol L7805CV -> SmartFan-rescue:L7805CV
- U2, U3, U4: symbol LTV-816S-TA1 -> SmartFan-rescue:LTV-816S-TA1
- U5: symbol LD1117S33CTR -> SmartFan-rescue:LD1117S33CTR
Connections:
- net labels added: +3V3, ANT_LED_OUT, BTLE_LED_OUT, MCP_INTA, MCP_INTA_5V, MCP_INTB, MCP_INTB_5V, RGB_G, RGB_G_OUT, RGB_R, RGB_R_OUT, RGB_Y, RGB_Y_OUT, SCL_3v3, SCL_5v, SDA_3v3, SDA_5v
- net labels removed: SPD_CTRL_PB
- wire segments 186 -> 299
- no-connect marks 36 -> 30
Other:
- note removed: "Fan Speed Control Pushbutton\n(Momentary)"

Commit message: swapped controller for hackaBLE module
Parts:
- removed C1: 10uF, Capacitors_SMD:C_0805, symbol SmartFan-rescue:C
- removed C5, C6: 1uF, Capacitors_SMD:C_0805, symbol SmartFan-rescue:C
- removed C7: 0.1uF, Capacitors_SMD:C_0805, symbol SmartFan-rescue:C
- removed D5: MBR0540T1G, digikey-footprints:SOD-123, symbol SmartFan-rescue:MBR0540T1G
- removed MOD1: BMD-300-A-R, digikey-footprints:Bluetooth_Module_BMD-300, symbol SmartFan-rescue:BMD-300-A-R
- removed R15, R19, R20: 330, Resistors_SMD:R_0805, symbol SmartFan-rescue:R
- removed U5: LD1117S33CTR, digikey-footprints:SOT-223, symbol SmartFan-rescue:LD1117S33CTR
- added J?: DISPLAY, Connectors_IDC:IDC-Header_2x10_Pitch2.54mm_Straight, symbol SmartFan-rescue:Conn_02x10_Odd_Even
- added U5: hackaBLE_0.3, symbol hackaBLE:hackaBLE_0.3
- gave numbers to parts that had none: 25
Connections:
- net +3V3: now also U5.16 (VDD), U5.22 (VDD)
- net +5V: now also J?.2 (Pin_2), U5.17 (VIN)
- net ANT_LED: now also U5.5 (P0.08)
- net ANT_LED_OUT: now also J?.12 (Pin_12)
- net BTLE_LED: now also U5.4 (P0.11)
- net BTLE_LED_OUT: now also J?.10 (Pin_10)
- net GND: now also J?.20 (Pin_20), U5.18 (GND), U5.21 (GND)
- net MCP_INTA: now also U5.6 (P0.07)
- net MCP_INTB: now also U5.7 (P0.06)
- net RGB_G: now also U5.3 (P0.12)
- net RGB_G_OUT: now also J?.4 (Pin_4)
- net RGB_R: now also U5.1 (P0.14)
- net RGB_R_OUT: now also J?.8 (Pin_8)
- net RGB_Y: now also U5.2 (P0.13)
- net RGB_Y_OUT: now also J?.6 (Pin_6)
- net SCL_3v3: now also U5.13 (P0.05)
- net SCL_5v: now also J?.3 (Pin_3)
- net SDA_3v3: now also U5.14 (P0.04)
- net SDA_5v: now also J?.1 (Pin_1)
- net SWCLK: now also U5.19 (SWDCLK)
- net SWDIO: now also U5.20 (SWDIO)
- net at R5.2: now also U5.10 (P0.27)
- net at R9.2: now also U5.11 (P0.26)
- net at R6.2: now also U5.12 (P0.25)
- net MCP_INTA_5V renamed MCP_INTA_5v
- net MCP_INTA_5v: now also J?.17 (Pin_17)
- net MCP_INTB_5V renamed MCP_INTB_5v
- net MCP_INTB_5v: now also J?.19 (Pin_19)
- net ~RESET: no longer names the net of J2.15 (Pin_15)
- no-connect marks 30 -> 14
Other:
- note added: "Display Board Port"
- note removed: "3.3v Power Regulator"
- moved on the sheet: C2, C3, C4, D1, D4, J1, J7, Q3, Q4, Q5, Q8, R10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

Commit message: mainboard updates
Parts:
- removed Q1, Q2: MMBT2222A-7-F, digikey-footprints:SOT-23-3, symbol SmartFan-rescue:MMBT2222A-7-F
- removed R1, R3: 220, Resistors_SMD:R_0805, symbol SmartFan-rescue:R
- removed R11, R21, R22: 220, symbol SmartFan-rescue:R
- removed R2, R4: 330, Resistors_SMD:R_0805, symbol SmartFan-rescue:R
- added U?: MCP23017_SP, Package_DIP:DIP-28_W7.62mm, symbol Interface_Expansion:MCP23017_SP
Connections:
- net RGB_G_OUT is gone; now on net RGB_G: J?.4 (Pin_4)
- net RGB_R_OUT is gone; now on net RGB_R: J?.8 (Pin_8)
- net RGB_Y_OUT is gone; now on net RGB_Y: J?.6 (Pin_6)
- net +5V: now also U?.10 (VSS), U?.18 (~RESET~), U?.9 (VDD)
- net ANT_LED: now also U?.25 (GPA4); no longer U5.5 (P0.08)
- net BTLE_LED: now also U?.24 (GPA3); no longer U5.4 (P0.11)
- net GND: now also U?.15 (A0), U?.16 (A1), U?.17 (A2)
- net MCP_INTA: now also U5.1 (P0.14); no longer U5.6 (P0.07)
- net MCP_INTA_5v: now also U?.19 (INTB)
- net MCP_INTB: now also U5.2 (P0.13); no longer U5.7 (P0.06)
- net RGB_G: now also U?.23 (GPA2); no longer U5.3 (P0.12)
- net RGB_R: now also U?.21 (GPA0); no longer U5.1 (P0.14)
- net RGB_Y: now also U?.22 (GPA1); no longer U5.2 (P0.13)
- net SCL_5v: now also U?.12 (SCK)
- net SDA_5v: now also U?.13 (SDA)
- new net MCB_INTB_5v: U?.20 (INTA)
- new net ROT_ENC_A: U?.1 (GPB0)
- new net ROT_ENC_B: U?.2 (GPB1)
- new net ROT_ENC_C: U?.3 (GPB2)
- new net ROT_ENC_SW1: U?.4 (GPB3)
- new net ROT_ENC_SW2: U?.5 (GPB4)
- no-connect marks 14 -> 19
Other:
- note removed: "ANT+ Indicator LED (Red)"
- note removed: "BTLE Indicator LED (Blue)"
- note removed: "Fan Speed Indicator LED"
- moved on the sheet: J2, J?, Q3, Q4, Q5, R10, R5, R6, R7, R8, R9, U5

Commit message: Remove relays and associated circuitry
Parts:
- removed D2, D3, D4: 1N4148W-7-F, digikey-footprints:SOD-123, symbol SmartFan-rescue:1N4148W-7-F
- removed J7: FAN_CONN, Connectors_Molex:Molex_MegaFit_2x02x5.70mm_Angled, symbol SmartFan-rescue:Conn_02x02_Counter_Clockwise
- removed Q3, Q4, Q5: MMBT2222A-TP, digikey-footprints:SOT-23-3, symbol SmartFan-rescue:MMBT2222A-TP
- removed Q6, Q7, Q8: MMBT2222A-7-F, digikey-footprints:SOT-23-3, symbol SmartFan-rescue:MMBT2222A-7-F
- removed R10, R7, R8: 10k, Resistors_SMD:R_0805, symbol SmartFan-rescue:R
- removed R12, R13, R14, R16, R17, R18, R5, R6, R9: 1k, Resistors_SMD:R_0805, symbol SmartFan-rescue:R
- removed RLY1, RLY2, RLY3: G5LE-14_DC5, digikey-footprints:Relay_THT_G5LE-14, symbol SmartFan-rescue:G5LE-14_DC5
- removed U2, U3, U4: LTV-816S-TA1, digikey-footprints:SMD-4_4.6x7.62mm_P2.54mm, symbol SmartFan-rescue:LTV-816S-TA1
- C2, C3, C4: symbol SmartFan-rescue:C -> SmartFan-rescue:C-SmartFan-rescue
- D1: symbol SmartFan-rescue:MBR0540T1G -> SmartFan-rescue:MBR0540T1G-SmartFan-rescue
- D5, D6: symbol SmartFan-rescue:1N914BTR -> SmartFan-rescue:1N914BTR-SmartFan-rescue
- J1: symbol SmartFan-rescue:Barrel_Jack -> SmartFan-rescue:Barrel_Jack-SmartFan-rescue
- J2, J?: symbol SmartFan-rescue:Conn_02x10_Odd_Even -> SmartFan-rescue:Conn_02x10_Odd_Even-SmartFan-rescue
- Q10, Q11, Q12, Q13, Q14, Q9: symbol SmartFan-rescue:2N3904 -> SmartFan-rescue:2N3904-SmartFan-rescue
- U1: symbol SmartFan-rescue:L7805CV -> SmartFan-rescue:L7805CV-SmartFan-rescue
- U5: symbol hackaBLE:hackaBLE_0.3 -> SmartFan-rescue:hackaBLE_0.3-hackaBLE
Connections:
- net HI_SPD_EN: now also U?.1 (GPB0)
- net LO_SPD_EN: now also U?.3 (GPB2)
- net MED_SPD_EN: now also U?.2 (GPB1)
- net ROT_ENC_A: now also U5.10 (P0.27); no longer U?.1 (GPB0)
- net ROT_ENC_B: now also U5.11 (P0.26); no longer U?.2 (GPB1)
- net ROT_ENC_C: now also U5.12 (P0.25); no longer U?.3 (GPB2)
- net ROT_ENC_SW1: now also U5.9 (P0.09); no longer U?.4 (GPB3)
- net ROT_ENC_SW2: now also U5.8 (P0.10); no longer U?.5 (GPB4)
- no-connect marks 19 -> 14
Other:
- moved on the sheet: U5
