File: hw/SmartFan.sch (KiCad schematic (older format))
At the start: 60 parts, among them J1 Barrel_Jack, J2 JTAG_SWD, J7 FAN_CONN, Q10 2N3904, Q11 2N3904, Q12 2N3904, Q13 2N3904, Q14 2N3904, Q3 MMBT2222A-TP, Q4 MMBT2222A-TP, Q5 MMBT2222A-TP, Q6 MMBT2222A-7-F, Q7 MMBT2222A-7-F, Q8 MMBT2222A-7-F, Q9 2N3904, U1 L7805CV, U2 LTV-816S-TA1, U3 LTV-816S-TA1, U4 LTV-816S-TA1, U5 hackaBLE_0.3

Commit message: Simplified schematic and pcb
Parts:
- removed D2, D3, D4: 1N4148W-7-F, digikey-footprints:SOD-123, symbol SmartFan-rescue:1N4148W-7-F
- removed J7: FAN_CONN, Connectors_Molex:Molex_MegaFit_2x02x5.70mm_Angled, symbol SmartFan-rescue:Conn_02x02_Counter_Clockwise
- removed Q10, Q11, Q12, Q14: 2N3904, TO_SOT_Packages_THT:TO-92_Molded_Narrow, symbol SmartFan-rescue:2N3904
- removed Q3, Q4, Q5: MMBT2222A-TP, digikey-footprints:SOT-23-3, symbol SmartFan-rescue:MMBT2222A-TP
- removed Q6, Q7, Q8: MMBT2222A-7-F, digikey-footprints:SOT-23-3, symbol SmartFan-rescue:MMBT2222A-7-F
- removed R10, R7, R8: 10k, Resistors_SMD:R_0805, symbol SmartFan-rescue:R
- removed R12, R13, R14, R16, R17, R18, R5, R6, R9: 1k, Resistors_SMD:R_0805, symbol SmartFan-rescue:R
- removed R24, R28, R30, R34: 330, symbol SmartFan-rescue:R
- removed R27, R29, R33, R36: R, symbol SmartFan-rescue:R
- removed RLY1, RLY2, RLY3: G5LE-14_DC5, digikey-footprints:Relay_THT_G5LE-14, symbol SmartFan-rescue:G5LE-14_DC5
- removed U2, U3, U4: LTV-816S-TA1, digikey-footprints:SMD-4_4.6x7.62mm_P2.54mm, symbol SmartFan-rescue:LTV-816S-TA1
- added J4: Relay_Terminal, TerminalBlock_RND:TerminalBlock_RND_205-00290_Pitch5.08mm, symbol Connector:Screw_Terminal_01x05
- C1: renamed from C2; footprint Capacitors_SMD:C_0805 -> Capacitors_THT:CP_Radial_D4.0mm_P1.50mm; DigikeyPN 1276-3010-1-ND -> 493-15541-ND
- C2: renamed from C3; footprint Capacitors_SMD:C_0805 -> Capacitors_THT:CP_Radial_D4.0mm_P1.50mm; DigikeyPN 1276-3010-1-ND -> 493-15541-ND
- C3: renamed from C4; footprint Capacitors_SMD:C_0805 -> Capacitors_THT:CP_Radial_D6.3mm_P2.50mm; DigikeyPN 1276-6840-1-ND -> 493-12624-1-ND
- D1: footprint digikey-footprints:SOD-123 -> digikey-footprints:DO-41; Digi-Key_PN MBR0540T1GOSCT-ND -> 1N5817FSCT-ND
- R1: renamed from R23; footprint (none) -> Resistors_THT:R_Axial_DIN0207_L6.3mm_D2.5mm_P10.16mm_Horizontal
- R2: renamed from R31; footprint (none) -> Resistors_THT:R_Axial_DIN0207_L6.3mm_D2.5mm_P10.16mm_Horizontal
- R3: renamed from R25; footprint (none) -> Resistors_THT:R_Axial_DIN0207_L6.3mm_D2.5mm_P10.16mm_Horizontal
- R4: renamed from R32; footprint (none) -> Resistors_THT:R_Axial_DIN0207_L6.3mm_D2.5mm_P10.16mm_Horizontal
- R5: renamed from R26; footprint (none) -> Resistors_THT:R_Axial_DIN0207_L6.3mm_D2.5mm_P10.16mm_Horizontal
- R6: renamed from R35; footprint (none) -> Resistors_THT:R_Axial_DIN0207_L6.3mm_D2.5mm_P10.16mm_Horizontal
- U1: renamed from U5; footprint (none) -> hackaBLE_0:hackaBLE_0.3
- U3: renamed from U?; footprint Package_DIP:DIP-28_W7.62mm -> Housings_DIP:DIP-28_W7.62mm_Socket
- gave numbers to parts that had none: 1
- renumbered D5 to D2, D6 to D3, J1 to J2, J2 to J3, Q9 to Q1, Q13 to Q2, U1 to U2
Connections:
- net labels removed: +3V3, 120VAC_IN, ANT_LED_OUT, BTLE_LED_OUT, HI_SPD_120VAC, LO_SPD_120VAC, MCB_INTB_5v, MCP_INTA, MCP_INTA_5v, MCP_INTB, MCP_INTB_5v, MED_SPD_120VAC, SCL_3v3, SDA_3v3
- wire segments 270 -> 141
- no-connect marks 19 -> 33
Other:
- moved on the sheet: C1, C2, C3, D1, D2, D3, J2, Q1, Q2, R1, R2, R3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

Commit message: Final v1 updates
Parts:
- added J3: PWR_SW, Connectors:PINHEAD1-2, symbol Connector:Conn_01x02_Male
- D1: footprint digikey-footprints:DO-41 -> Digikey:DO-41
- D2, D3: footprint digikey-footprints:DO-35 -> Digikey:DO-35
- J2: footprint Connectors:BARREL_JACK -> Connector_BarrelJack:BarrelJack_Horizontal
- U2: footprint digikey-footprints:SOT-23-3 -> Digikey:SOT-23-3
- renumbered J3 to J4, J4 to J5
Connections:
- net +9V: now also J3.2 (Pin_2); no longer C1.1, U2.1 (IN)
- net SCL_5v: no longer J1.3 (Pin_3)
- net SDA_5v: no longer J1.1 (Pin_1)
- net SCL_3v3: now reaches D2.A, Q1.1 (E), R1.2, U1.13 (P0.05)
- net SCL_3v3: now also J1.3 (Pin_3)
- net SDA_3v3: now reaches D3.A, Q2.1 (E), R2.2, U1.14 (P0.04)
- net SDA_3v3: now also J1.1 (Pin_1)
- new net: C1.1, J3.1 (Pin_1), U2.1 (IN)
Other:
- moved on the sheet: C1, C2, C3, D1, U2

Commit message: Hardware design updates
Parts:
- removed J2: Barrel_Jack, Connector_BarrelJack:BarrelJack_Horizontal, symbol SmartFan-rescue:Barrel_Jack
- added J2: PJ-102A, digikey-footprints:Barrel_Jack_5.5mmODx2.1mmID_PJ-102A, symbol dk_Barrel-Power-Connectors:PJ-102A
- C1, C2: footprint Capacitors_THT:CP_Radial_D4.0mm_P1.50mm -> Capacitor_THT:CP_Radial_D4.0mm_P1.50mm
- C3: footprint Capacitors_THT:CP_Radial_D6.3mm_P2.50mm -> Capacitor_THT:CP_Radial_D6.3mm_P2.50mm
- D1: footprint Digikey:DO-41 -> digikey-footprints:DO-41
- D2, D3: footprint Digikey:DO-35 -> digikey-footprints:DO-35
- J1, J4: footprint Connectors_IDC:IDC-Header_2x10_Pitch2.54mm_Straight -> Connector_IDC:IDC-Header_2x10_P2.54mm_Vertical
- J3: footprint Connectors:PINHEAD1-2 -> Connector_PinHeader_2.54mm:PinHeader_1x02_P2.54mm_Vertical
- J5: footprint TerminalBlock_RND:TerminalBlock_RND_205-00290_Pitch5.08mm -> TerminalBlock_RND:TerminalBlock_RND_205-00290_1x05_P5.08mm_Horizontal
- Q1, Q2: footprint TO_SOT_Packages_THT:TO-92_Molded_Narrow -> digikey-footprints:TO-92-3
- R1, R2, R3, R4, R5, R6: footprint Resistors_THT:R_Axial_DIN0207_L6.3mm_D2.5mm_P10.16mm_Horizontal -> Resistor_THT:R_Axial_DIN0207_L6.3mm_D2.5mm_P10.16mm_Horizontal
- U2: footprint Digikey:SOT-23-3 -> digikey-footprints:SOT-23-3
- U3: footprint Housings_DIP:DIP-28_W7.62mm_Socket -> digikey-footprints:Socket_DIP-28_7.62mm_Conn
Connections:
- net +5V: no longer U3.10 (VSS)
- net +9V: now also J2.2
- net GND: now also U3.10 (VSS), J2.1

Commit message: updates
Connections:
- net SCL_3v3: no longer J1.3 (Pin_3)
- net SDA_3v3: no longer J1.1 (Pin_1)
- net SDI_MOSI: now reaches U1.1 (P0.14)
- net SDI_MOSI: now also J1.1 (Pin_1)
- net SDI_MISO: now reaches U1.2 (P0.13)
- net SDI_MISO: now also J1.3 (Pin_3)
- net SDI_SCK: now reaches U1.3 (P0.12)
- net SDI_SCK: now also J1.5 (Pin_5)
- net SDI_DC_RS: now reaches U1.4 (P0.11)
- net SDI_DC_RS: now also J1.7 (Pin_7)
- net SDI_CS_LCD: now reaches U1.5 (P0.08)
- net SDI_CS_LCD: now also J1.14 (Pin_14)
- net SDI_CS_TS: now reaches U1.6 (P0.07)
- net SDI_CS_TS: now also J1.16 (Pin_16)
- net IRQ_TS: now reaches U1.7 (P0.06)
- net IRQ_TS: now also J1.18 (Pin_18)
- no-connect marks 33 -> 21
Changed lines of the file:
@@
 EESchema Schematic File Version 4
 LIBS:SmartFan-cache
-EELAYER 26 0
+EELAYER 30 0
 EELAYER END
 $Descr B 17000 11000
@@
 ANT_LED
 Wire Wire Line
-	1250 8950 700  8950
-Wire Wire Line
 	1250 9050 700  9050
 $Comp
@@
 Wire Wire Line
 	11750 5750 12300 5750
-NoConn ~ 2850 4850
-NoConn ~ 2850 4950
-NoConn ~ 2850 5050
 Wire Notes Line
 	2650 10400 2650 8300
@@
 Wire Wire Line
 	2750 9300 3450 9300
-NoConn ~ 2850 4650
-NoConn ~ 2850 4750
 Wire Wire Line
 	4050 4450 4600 4450
@@
 Wire Wire Line
 	6350 4850 6350 6450
-NoConn ~ 1250 9150
-NoConn ~ 1250 9250
 Text Label 8900 4450 0    50   ~ 0
 SDA_5v
 Text Label 8900 4750 0    50   ~ 0
 SCL_5v
-NoConn ~ 1750 9750
-NoConn ~ 1750 9650
-NoConn ~ 1750 9550
 NoConn ~ 1250 9850
-NoConn ~ 2850 4450
-NoConn ~ 2850 4550
 $Comp
 L SmartFan-rescue:Conn_02x10_Odd_Even J1
@@
 Text Label 4600 4850 2    50   ~ 0
 SDA_3v3
-Text Label 700  8950 0    50   ~ 0
-SDA_3v3
-Text Label 700  9050 0    50   ~ 0
-SCL_3v3
 $Comp
 L dk_Barrel-Power-Connectors:PJ-102A J2
@@
 Wire Wire Line
 	10500 6550 11050 6550
+Wire Wire Line
+	1250 8950 700  8950
+Wire Wire Line
+	1250 9150 700  9150
+Text Label 700  8950 0    50   ~ 0
+SDI_MOSI
+Text Label 700  9050 0    50   ~ 0
+SDI_MISO
+Text Label 700  9150 0    50   ~ 0
+SDI_SCK
+Wire Wire Line
+	1750 9650 2350 9650
+Wire Wire Line
+	1750 9750 2350 9750
+Wire Wire Line
+	1250 9250 700  9250
+Text Label 700  9250 0    50   ~ 0
+SDI_DC_RS
+Text Label 2350 9550 2    50   ~ 0
+SDI_CS_LCD
+Text Label 2350 9650 2    50   ~ 0
+SDI_CS_TS
+Wire Wire Line
+	1750 9550 2350 9550
+Text Label 2350 9750 2    50   ~ 0
+IRQ_TS
+Wire Wire Line
+	2850 4450 2100 4450
+Wire Wire Line
+	2850 4550 2100 4550
+Wire Wire Line
+	2850 4650 2100 4650
+Wire Wire Line
+	2850 4750 2100 4750
+Wire Wire Line
+	2850 4850 2100 4850
+Wire Wire Line
+	2850 4950 2100 4950
+Wire Wire Line
+	2850 5050 2100 5050
+Text Label 2100 4450 0    50   ~ 0
+SDI_MOSI
+Text Label 2100 4550 0    50   ~ 0
+SDI_MISO
+Text Label 2100 4650 0    50   ~ 0
+SDI_SCK
+Text Label 2100 4750 0    50   ~ 0
+SDI_DC_RS
+Text Label 2100 4850 0    50   ~ 0
+SDI_CS_LCD
+Text Label 2100 4950 0    50   ~ 0
+SDI_CS_TS
+Text Label 2100 5050 0    50   ~ 0
+IRQ_TS
 $EndSCHEMATC
